File: Processing_board/ADC 2.kicad_sch (KiCad schematic)
At the start: 58 parts, among them U10 ADS1299IPAG, U11 ADS1299IPAG

Commit message: feat: bias network, GPIO
Parts:
- R11, R12, R22, R23, R24, R25, R26, R27, R28: value 47kΩ -> ?
Connections:
- net CS1: no longer names the net of U10.39 (*CS)
- net CS2: no longer names the net of U11.39 (*CS)
- net DRDY: no longer names the net of U10.47 (*DRDY)
- net DRDY: no longer U11.47 (*DRDY)
- net MISO: no longer names the net of U10.43 (DOUT)
- net MISO: no longer U11.43 (DOUT)
- net MOSI: no longer names the net of U10.34 (DIN)
- net MOSI: no longer U11.34 (DIN)
- net PWDN: no longer names the net of U10.35 (*PWDN)
- net PWDN: no longer U11.35 (*PWDN)
- net RESET: no longer names the net of U10.36 (*RESET)
- net RESET: no longer U11.36 (*RESET)
- net SCK: no longer names the net of U10.40 (SCLK)
- net SCK: no longer U11.40 (SCLK)
- no-connect marks 16 -> 4
